File: narsil.brd (EAGLE design)
At the start: 160 x 120.3 mm, 18 parts, among them U1 STM32F10XRXT6, X1 PN61729-S

Commit message: Schematic ready
Parts:
- added ANALOG_LDO, DIGITAL_LDO: ADP3335ARM-3.3RL7, analog-devices:MSOP08
- added BTN_0, BTN_1, BTN_2, RESET: 10-XXG, switch-omron:B3F-10XXG
- added C10, C16, C28, C33, C35, C8, C9: (no value), resistor:SMC_A
- added C11, C12, C13, C41, C42, C43, C44, C7: (no value), resistor:C0805
- added C14, C26: 100n, rcl:C0805
- added C15, C27: 100u, rcl:C0805
- added C32, C34: 100n, resistor:C0805
- added D1, D3: (no value), diode:SMB
- added JP1, JP7: (no value), jumper:JP1
- added JTAG: (no value), jumper:JP5Q
- added L2, L3: (no value), resistor:R1206
- added LED_0, LED_1, LED_PWR: (no value), led:1206
- added Q1, Q5: IRLML5203, transistor-power:MICRO3
- added R1, R10, R11, R13, R34, R35, R36, R37: 5k, resistor:M0805
- added R12, R7: 10K, resistor:M0805
- added R2, R3, R4, R5, R6, R8, R9: 47k, resistor:M0805
- added SPI2: 22-23-2051, con-molex:22-23-2051
- added U$1: SD-RSMT-2-MQ, SD-RSMT-2-MQ:SD-RSMT-2-MQ
- added U$2: LCD, nokia_lcd:LCD_NOKIA1100
- added UART1: (no value), jumper:JP4
- moved X1 32.5 mm to (40.6, 66.0)
- moved ADC0 10.5 mm to (109.2, 33.0)
- moved ADC1 10.5 mm to (109.2, 48.3)
- moved ADC2 10.5 mm to (109.2, 63.5)
- moved ADC3 10.5 mm to (109.2, 78.7)
- moved APWR 10.5 mm to (109.2, 17.8)
- moved QF1 9.25 mm to (78.7, 26.7)
- moved U1 7.41 mm to (80.0, 44.5)
Connections:
- new net +5V: C32.1, C35.+, D3.A, L2.1, X1.1
- new net A6: U1.22
- new net N$14: R9.1, X1.2
- new net N$15: LED_1.A, R11.2
- new net N$16: R8.1, X1.3
- new net N$17: LED_0.A, R13.2
- new net N$18: U$1.WP
- new net N$19: U$1.CD
- new net N$20: D3.C, JP7.2
- new net N$21: ANALOG_LDO.6, ANALOG_LDO.7, ANALOG_LDO.8, C14.1, JP1.1
- new net N$22: D1.C, JP1.2
- new net N$23: C33.+, C34.1, D1.A, L2.2
- new net N$28: C41.2, JTAG.6, R34.2, RESET.3, RESET.4, U1.7
- new net N$32: C26.1, DIGITAL_LDO.6, DIGITAL_LDO.7, DIGITAL_LDO.8, JP7.1
- new net PA10: U1.43, UART1.1
- new net PA11: C12.1, R9.2, U1.44
- new net PA12: C13.1, Q1.2, R8.2, U1.45
- new net PA13: JTAG.5, U1.46
- new net PA14: JTAG.1, U1.49
- new net PA15: JTAG.9, U1.50
- new net PA7: U1.23
- new net PA8: U1.41, UART1.3
- new net PA9: U1.42, UART1.2
- new net PB0: U1.26
- new net PB1: U1.27
- new net PB10: U$2.P$4, U1.29
- new net PB11: U$2.P$5, U1.30
- new net PB12: SPI2.4, U1.33
- new net PB13: SPI2.3, U1.34
- new net PB14: SPI2.2, U1.35
- new net PB15: SPI2.1, U1.36
- new net PB2: Q5.1, R12.2, U1.28
- new net PB3: JTAG.3, U1.55
- new net PB4: JTAG.8, U1.56
- new net PB5: LED_0.C, U1.57
- new net PB6: LED_1.C, U1.58
- new net PB7: Q1.1, R7.1, U1.59
- new net PB8: U$2.P$1, U1.61
- new net PB9: U$2.P$2, U1.62
- new net PC0: U1.8
- new net PC1: U1.9
- new net PC10: R4.1, U$1.9, U1.51
- new net PC11: R2.1, U$1.1, U1.52
- new net PC12: U$1.5, U1.53
- new net PC13: BTN_0.3, BTN_0.4, C44.2, R37.2, U1.2
- new net PC14: BTN_1.3, BTN_1.4, C43.2, R36.2, U1.3
- new net PC15: BTN_2.3, BTN_2.4, C42.2, R35.2, U1.4
- new net PC2: U1.10
- new net PC3: U1.11
- new net PC4: U1.24
- new net PC5: U1.25
- new net PC6: U1.37
- new net PC7: U1.38
- new net PC8: R6.1, U$1.7, U1.39
- new net PC9: R5.1, U$1.8, U1.40
- new net PD2: R3.1, U$1.2, U1.54
- net AGND: now also ADC0.2, ADC1.2, ADC2.2, ADC3.2, ANALOG_LDO.4, C10.-, C14.2, C15.2, C16.-, C33.-, C34.2, DAC1.2, DAC2.2, L3.2
- net GND: now also BTN_0.1, BTN_0.2, BTN_0.G, BTN_1.1, BTN_1.2, BTN_1.G, BTN_2.1, BTN_2.2, BTN_2.G, C12.2, C13.2, C26.2, C27.2, C28.-, C32.2, C35.-, C41.1, C42.1, C43.1, C44.1, C7.1, C8.-, C9.-, DIGITAL_LDO.4, JTAG.10, JTAG.2, JTAG.4, L3.1, LED_PWR.C, R1.1, RESET.1, RESET.2, RESET.G, SPI2.5, U$1.3, U$1.6, U$1.GP, U$1.GP2, U$2.P$3, UART1.4, X1.4, X1.SHLD@1, X1.SHLD@2; no longer ADC0.2, ADC1.2, ADC2.2, DAC1.2, DAC2.2
- net N$11: now also R1.2, U1.60; no longer ADC3.2
- net N$12: now also Q5.3, U$2.P$8; no longer U1.45, X1.3
- net N$13: now also LED_PWR.A, R10.2; no longer U1.44, X1.2
- net VCC: now also C27.1, C28.+, C7.2, C8.+, C9.+, DIGITAL_LDO.1, DIGITAL_LDO.2, DIGITAL_LDO.3, JTAG.7, Q1.3, Q5.2, R10.1, R11.1, R12.1, R13.1, R2.2, R3.2, R34.1, R35.1, R36.1, R37.1, R4.2, R5.2, R6.2, R7.2, U$1.4, U$2.P$6, U$2.P$7
- net VDD: now also ANALOG_LDO.1, ANALOG_LDO.2, ANALOG_LDO.3, C10.+, C11.1, C15.1, C16.+
Other:
- board size 160 x 120.3 mm -> 222.2 x 75.9 mm

Commit message: layout is close to ready: there is no LCD only
Parts:
- removed C10: (no value), resistor:SMC_A
- removed JP7: (no value), jumper:JP1
- QF1: value 10M15AHC49T -> ACT530SMX; device crystal:HC49U -> crystal:ACT530SMX
- moved JTAG 437.7 mm to (49.5, 82.0)
- moved C33 397.5 mm to (90.8, 23.2), turned to 90 degrees
- moved C16 393.0 mm to (95.8, 35.4), turned to 180 degrees
- moved L2 390.6 mm to (85.4, 22.3)
- moved L3 390.1 mm to (85.4, 24.4)
- moved C35 390.0 mm to (80.0, 23.3), turned to 90 degrees
- moved C15 389.1 mm to (95.7, 33.6), turned to 180 degrees
- moved C34 384.6 mm to (89.0, 23.2), turned to 90 degrees
- moved C32 384.3 mm to (81.8, 23.3), turned to 90 degrees
- moved ANALOG_LDO 379.3 mm to (95.8, 29.3), turned to 180 degrees
- moved D1 377.1 mm to (95.1, 23.3), turned to 180 degrees
- moved JP1 367.6 mm to (78.0, 13.3), turned to 90 degrees
- moved C14 360.8 mm to (92.9, 27.1), turned to 90 degrees
- moved C28 344.6 mm to (79.8, 21.8), flipped to the bottom, turned to 270 degrees
- moved C27 341.5 mm to (77.8, 21.8), flipped to the bottom, turned to 270 degrees
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Connections:
- removed net N$22: D1.C, JP1.2
- removed net VBAT: U1.1
- net AGND: now also C11.2; no longer C10.-
- net GND: now also JP1.2, QF1.S$1, QF1.S$2; no longer QF1.2
- net N$20: now also JP1.1, U1.1; no longer D3.C, JP7.2
- net N$21: now also D1.C; no longer JP1.1
- net N$3: now also QF1.P2; no longer QF1.3
- net N$32: now also D3.C; no longer JP7.1
- net N$4: now also QF1.P1; no longer QF1.1
- net VDD: no longer C10.+
Routing:
- net GND: track 0.00 -> 271.2 mm, vias 0 -> 1
- net VCC: track 0.00 -> 216.2 mm, vias 0 -> 4
- net N$28: track 0.00 -> 131.0 mm
- net PB4: track 0.00 -> 97.3 mm
- net +5V: track 0.00 -> 95.2 mm, vias 0 -> 1
- net PB7: track 0.00 -> 78.7 mm
- net PB3: track 0.00 -> 77.6 mm
- net PA15: track 0.00 -> 69.7 mm
- net PC13: track 0.00 -> 64.5 mm
- net PB6: track 0.00 -> 59.3 mm, vias 0 -> 2
- net PB9: track 0.00 -> 59.1 mm
- net PB8: track 0.00 -> 58.1 mm
- net PB5: track 0.00 -> 55.5 mm, vias 0 -> 2
- net PC14: track 0.00 -> 54.7 mm
- net PA8: track 0.00 -> 53.5 mm
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- added copper zone on layer 1, net AGND
- added copper zone on layer 16, net AGND
- added copper zone on layer 1, net GND
- added copper zone on layer 16, net GND
- added copper zone on layer 1, net N$22

Commit message: v0.4 OK
Parts:
- moved C3 31.0 mm to (48.0, 32.2), turned to 180 degrees
- moved Q5 30.7 mm to (16.0, 47.6), turned to 180 degrees
- moved X1 30.3 mm to (8.14, 68.3)
- moved C1 29.9 mm to (51.2, 39.4), turned to 270 degrees
- moved C14 28.7 mm to (66.0, 17.0)
- moved C15 28.7 mm to (68.9, 23.5)
- moved C32 28.7 mm to (54.9, 13.1)
- moved C6 28.7 mm to (61.7, 24.9)
- moved DAC1 28.7 mm to (67.1, 68.6)
- moved R5 28.7 mm to (39.3, 19.0)
- moved R6 28.7 mm to (39.3, 21.5)
- moved U1 28.7 mm to (53.2, 34.3)
- moved BTN_2 28.7 mm to (30.0, 5.96)
- moved C11 28.7 mm to (59.7, 30.6)
- moved C26 28.7 mm to (43.4, 15.1)
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Routing:
- net GND: track 271.2 -> 38.3 mm, vias 1 -> 13
- net VCC: track 216.2 -> 279.5 mm, vias 4 -> 8
- net PB2: track 0.00 -> 54.6 mm, vias 0 -> 4
- net PB11: track 0.43 -> 52.6 mm, vias 0 -> 4
- net PB10: track 0.00 -> 44.8 mm, vias 0 -> 2
- net +5V: track 95.2 -> 105.7 mm
- net N$14: track 2.34 -> 9.24 mm
- net N$13: track 0.00 -> 5.33 mm, vias 0 -> 1
- net PA15: track 69.7 -> 74.6 mm
- net PA14: track 50.9 -> 55.4 mm
- net PB7: track 78.7 -> 82.8 mm, vias 0 -> 1
- net PB9: track 59.1 -> 62.4 mm
- net PA11: track 47.4 -> 44.6 mm
- net PA12: track 49.8 -> 46.9 mm
- net PA13: track 46.8 -> 49.4 mm
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- removed copper zone on layer 1, net N$22
Other:
- board size 222.2 x 75.9 mm -> 90 x 75 mm
- board text added: "Narsil"
- board text added: "goron.dekar@gmail.com"
- board text added: "v0.4"

Commit message: v0.5
Parts:
- added JP2: (no value), jumper:JP1
- added JP3, JP4: (no value), jumper:JP4
- moved JP1 3.90 mm to (51.0, 7.10)
Connections:
- net GND: now also JP2.2
- net PC0: now also JP3.4
- net PC1: now also JP3.3
- net PC2: now also JP3.2
- net PC3: now also JP3.1
- net PC4: now also JP4.4
- net PC5: now also JP4.3
- net VCC: now also JP2.1
Routing:
- net PC4: track 0.00 -> 39.7 mm
- net PC5: track 0.00 -> 38.8 mm
- net PC0: track 0.00 -> 20.3 mm
- net PC1: track 0.00 -> 18.4 mm
- net PC2: track 0.00 -> 16.5 mm
- net PC3: track 0.00 -> 14.7 mm
- net VCC: track 279.5 -> 285.9 mm
- net N$5: track 30.2 -> 35.7 mm
- net N$6: track 39.8 -> 44.3 mm
- net N$20: track 29.1 -> 25.6 mm
- net N$8: track 33.9 -> 35.4 mm
- net AGND: vias 3 -> 7
Other:
- board text added: "v0.5"
- board text removed: "v0.4"

Commit message: v0.6
Parts:
- added C21, C22: (no value), resistor:C0805
- added Q2: 32kHz, crystal:MC146
- added R/C3: (no value), resistor:M0805
- moved C11 2.19 mm to (61.9, 30.6), turned to 180 degrees
- moved C2 1.97 mm to (52.3, 31.3), turned to 180 degrees
- moved R/C2 0.75 mm to (50.1, 34.7)
Connections:
- new net N$22: R/C3.2, U1.6
- net GND: now also C21.1, C22.1, Q2.GND, Q2.GND2
- net N$4: now also R/C3.1; no longer U1.6
- net PC14: now also C21.2, Q2.P$1; no longer BTN_1.3, BTN_1.4, C43.2, R36.2
- net PC15: now also C22.2, Q2.P$2; no longer BTN_2.3, BTN_2.4, C42.2, R35.2
- net PC6: now also BTN_2.3, BTN_2.4, C42.2, R35.2
- net PC7: now also BTN_1.3, BTN_1.4, C43.2, R36.2
Routing:
- net PC6: track 0.00 -> 68.4 mm, vias 0 -> 4
- net PC7: track 0.00 -> 67.7 mm, vias 0 -> 4
- net PC14: track 54.2 -> 9.87 mm, vias 0 -> 1
- net PC15: track 51.2 -> 13.0 mm, vias 0 -> 1
- net AGND: track 11.5 -> 7.77 mm
- net N$22: track 0.00 -> 3.20 mm, vias 0 -> 1
- net N$28: track 133.5 -> 135.9 mm
- net PC13: track 64.3 -> 66.5 mm
- net VDD: track 49.5 -> 48.1 mm
- net VCC: track 285.9 -> 287.0 mm
- net N$4: track 8.41 -> 8.64 mm, vias 0 -> 1
- net GND: track 38.3 -> 38.1 mm, vias 13 -> 14
Other:
- board text added: "v0.6"
- board text removed: "v0.5"
