File: narsil.sch (EAGLE design)
At the start: 18 parts, among them U1 STM32F10XRXT6, X1 PN61729-S

Commit message: Schematic ready
Parts:
- added ANALOG_LDO, DIGITAL_LDO: ADP3335ARM-3.3RL7, analog-devices:ADP3335ARM-3.3RL7
- added BTN_0, BTN_1, BTN_2, RESET: 10-XXG, switch-omron:10-XXG
- added C10, C16, C28, C33, C35, C8, C9: (no value), resistor:CPOL-EUSMCA
- added C11, C12, C13, C41, C42, C43, C44, C7: (no value), resistor:C-EUC0805
- added C14, C26: 100n, rcl:C-EUC0805
- added C15, C27: 100u, rcl:C-EUC0805
- added C32, C34: 100n, resistor:C-EUC0805
- added D1, D3: (no value), diode:ZENER-DIODESMB
- added JP1, JP7: (no value), jumper:JP1E
- added JTAG: (no value), jumper:JP5Q
- added L2, L3: (no value), resistor:L-EUL1206
- added LED_0, LED_1, LED_PWR: (no value), led:LEDSMT1206
- added Q1, Q5: IRLML5203, transistor-power:IRLML5203
- added R1, R10, R11, R13, R34, R35, R36, R37: 5k, resistor:R-EU_M0805
- added R12, R7: 10K, resistor:R-EU_M0805
- added R2, R3, R4, R5, R6, R8, R9: 47k, resistor:R-EU_M0805
- added SPI2: 22-23-2051, con-molex:22-23-2051
- added U$1: SD-RSMT-2-MQ, SD-RSMT-2-MQ:SD-RSMT-2-MQ
- added U$2: LCD, nokia_lcd:LCD
- added UART1: (no value), jumper:JP4E
Connections:
- new net +5V: C32.1, C35.+, D3.A, L2.1, X1.1
- new net A6: U1PORTA_L.PA6
- new net N$14: R9.1, X1.2
- new net N$15: LED_1.A, R11.2
- new net N$16: R8.1, X1.3
- new net N$17: LED_0.A, R13.2
- new net N$18: U$1.WRITE_PROTECT
- new net N$19: U$1.CARD_DETECT
- new net N$20: D3.C, JP7.2
- new net N$21: ANALOG_LDO.IN, ANALOG_LDO.IN@1, ANALOG_LDO.SD/, C14.1, JP1.1
- new net N$22: D1.C, JP1.2
- new net N$23: C33.+, C34.1, D1.A, L2.2
- new net N$28: C41.2, JTAG.6, R34.2, RESET.S, RESET.S1, U1RESET.NRST
- new net N$32: C26.1, DIGITAL_LDO.IN, DIGITAL_LDO.IN@1, DIGITAL_LDO.SD/, JP7.1
- new net PA10: U1PORTA_H.PA10, UART1.1
- new net PA11: C12.1, R9.2, U1PORTA_H.PA11
- new net PA12: C13.1, Q1.S, R8.2, U1PORTA_H.PA12
- new net PA13: JTAG.5, U1PORTA_H.PA13
- new net PA14: JTAG.1, U1PORTA_H.PA14
- new net PA15: JTAG.9, U1PORTA_H.PA15
- new net PA7: U1PORTA_L.PA7
- new net PA8: U1PORTA_H.PA8, UART1.3
- new net PA9: U1PORTA_H.PA9, UART1.2
- new net PB0: U1PORTB_L.PB0
- new net PB1: U1PORTB_L.PB1
- new net PB10: U$2.SDA, U1PORTB_H.PB10
- new net PB11: U$2.SCLK, U1PORTB_H.PB11
- new net PB12: SPI2-4.S, U1PORTB_H.PB12
- new net PB13: SPI2-3.S, U1PORTB_H.PB13
- new net PB14: SPI2-2.S, U1PORTB_H.PB14
- new net PB15: SPI2-1.S, U1PORTB_H.PB15
- new net PB2: Q5.G, R12.2, U1PORTB_L.PB2
- new net PB3: JTAG.3, U1PORTB_L.PB3
- new net PB4: JTAG.8, U1PORTB_L.PB4
- new net PB5: LED_0.C, U1PORTB_L.PB5
- new net PB6: LED_1.C, U1PORTB_L.PB6
- new net PB7: Q1.G, R7.1, U1PORTB_L.PB7
- new net PB8: U$2.XRES, U1PORTB_H.PB8
- new net PB9: U$2.XCS, U1PORTB_H.PB9
- new net PC0: U1PORTC_L.PC0
- new net PC1: U1PORTC_L.PC1
- new net PC10: R4.1, U$1.DAT2, U1PORTC_H.PC10
- new net PC11: R2.1, U$1.DAT3, U1PORTC_H.PC11
- new net PC12: U$1.SCLK, U1PORTC_H.PC12
- new net PC13: BTN_0.S, BTN_0.S1, C44.2, R37.2, U1PORTC_H.PC13
- new net PC14: BTN_1.S, BTN_1.S1, C43.2, R36.2, U1PORTC_H.PC14
- new net PC15: BTN_2.S, BTN_2.S1, C42.2, R35.2, U1PORTC_H.PC15
- new net PC2: U1PORTC_L.PC2
- new net PC3: U1PORTC_L.PC3
- new net PC4: U1PORTC_L.PC4
- new net PC5: U1PORTC_L.PC5
- new net PC6: U1PORTC_L.PC6
- new net PC7: U1PORTC_L.PC7
- new net PC8: R6.1, U$1.DAT0, U1PORTC_H.PC8
- new net PC9: R5.1, U$1.DAT1, U1PORTC_H.PC9
- new net PD2: R3.1, U$1.CMD, U1PORTD/OSC.PD2
- net AGND: now also ADC0.GND, ADC1.GND, ADC2.GND, ADC3.GND, ANALOG_LDO.GND, C10.-, C14.2, C15.2, C16.-, C33.-, C34.2, DAC1.GND, DAC2.GND, L3.2
- net GND: now also BTN_0.GND, BTN_0.P, BTN_0.P1, BTN_1.GND, BTN_1.P, BTN_1.P1, BTN_2.GND, BTN_2.P, BTN_2.P1, C12.2, C13.2, C26.2, C27.2, C28.-, C32.2, C35.-, C41.1, C42.1, C43.1, C44.1, C7.1, C8.-, C9.-, DIGITAL_LDO.GND, JTAG.10, JTAG.2, JTAG.4, L3.1, LED_PWR.C, R1.1, RESET.GND, RESET.P, RESET.P1, SPI2-5.S, U$1.SHLD, U$1.VSS1, U$1.VSS2, U$2.GND, UART1.4, X1.4, X1.S1
- net N$11: now also R1.2, U1RESET.BOOT0; no longer ADC3.GND
- net N$12: now also Q5.D, U$2.LED; no longer U1PORTA_H.PA12, X1.3
- net N$13: now also LED_PWR.A, R10.2; no longer U1PORTA_H.PA11, X1.2
- net VCC: now also C27.1, C28.+, C7.2, C8.+, C9.+, DIGITAL_LDO.OUT, DIGITAL_LDO.OUT@1, DIGITAL_LDO.OUT@2, JTAG.7, Q1.D, Q5.S, R10.1, R11.1, R12.1, R13.1, R2.2, R3.2, R34.1, R35.1, R36.1, R37.1, R4.2, R5.2, R6.2, R7.2, U$1.VDD, U$2.VDD, U$2.VDDI
- net VDD: now also ANALOG_LDO.OUT, ANALOG_LDO.OUT@1, ANALOG_LDO.OUT@2, C10.+, C11.1, C15.1, C16.+
Other:
- note added: "CK"
- note added: "D+"
- note added: "D-"
- note added: "GND"
- note added: "LCD"
- note added: "MISO"
- note added: "MOSI"
- note added: "NSRST"
- note added: "NSS"
- note added: "NTRST"
- note added: "RX"
- note added: "SCK"
- note added: "TCK"
- note added: "TDI"
- note added: "TDO"
- note added: "TMS"
- note added: "TX"
- note added: "VCC"
- moved on the sheet: ADC0, ADC1, ADC2, ADC3, APWR, C1, C2, C3, C4, C5, C6, DAC1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

Commit message: layout is close to ready: there is no LCD only
Parts:
- removed C10: (no value), resistor:CPOL-EUSMCA
- removed JP7: (no value), jumper:JP1E
- QF1: value 10M15AHC49T -> ACT530SMX; device crystal:10M15AHC49T -> crystal:ACT530SMX
Connections:
- removed net N$22: D1.C, JP1.2
- net AGND: now also C11.2; no longer C10.-
- net GND: now also JP1.2
- net N$20: now also JP1.1, U1AN_POWER.VBAT; no longer D3.C, JP7.2
- net N$21: now also D1.C; no longer JP1.1
- net N$32: now also D3.C; no longer JP7.1
- net VDD: no longer C10.+
Other:
- moved on the sheet: JP1
Changed lines of the file:
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@@
 <part name="C4" library="resistor" deviceset="C-EU" device="C0805"/>
 <part name="GND5" library="supply1" deviceset="GND" device=""/>
-<part name="QF1" library="crystal" deviceset="10M*A" device="HC49T" technology="15"/>
+<part name="QF1" library="crystal" deviceset="ACT530SMX" device=""/>
 <part name="C5" library="resistor" deviceset="C-EU" device="C0805"/>
 <part name="C6" library="resistor" deviceset="C-EU" device="C0805"/>
@@
 <part name="R6" library="resistor" deviceset="R-EU_" device="M0805" value="47k"/>
 <part name="C9" library="resistor" deviceset="CPOL-EU" device="SMCA"/>
-<part name="C10" library="resistor" deviceset="CPOL-EU" device="SMCA"/>
 <part name="C11" library="resistor" deviceset="C-EU" device="C0805"/>
 <part name="P+5" library="supply1" deviceset="VCC" device=""/>
@@
 <part name="P+11" library="supply1" deviceset="VCC" device=""/>
 <part name="C28" library="resistor" deviceset="CPOL-EU" device="SMCA"/>
-<part name="JP7" library="jumper" deviceset="JP1E" device=""/>
 <part name="D3" library="diode" deviceset="ZENER-DIODE" device="SMB"/>
 <part name="P+10" library="supply1" deviceset="+5V" device=""/>
@@
 <part name="ANALOG_LDO" library="analog-devices" deviceset="ADP3335ARM-3.3" device="RL7"/>
 <part name="C16" library="resistor" deviceset="CPOL-EU" device="SMCA"/>
-<part name="JP1" library="jumper" deviceset="JP1E" device=""/>
 <part name="D1" library="diode" deviceset="ZENER-DIODE" device="SMB"/>
 <part name="P+14" library="supply1" deviceset="+5V" device=""/>
@@
 <part name="P+13" library="supply1" deviceset="VCC" device=""/>
 <part name="GND12" library="supply1" deviceset="GND" device=""/>
+<part name="JP1" library="jumper" deviceset="JP1E" device=""/>
+<part name="GND13" library="supply1" deviceset="GND" device=""/>
 </parts>
 <sheets>
@@
 <attribute name="VALUE" x="40.1574" y="257.937" size="1.778" layer="96" rot="MR270"/>
 </instance>
-<instance part="C10" gate="G$1" x="40.64" y="165.1" smashed="yes" rot="MR0">
-<attribute name="NAME" x="44.9834" y="168.021" size="1.778" layer="95" rot="MR270"/>
-<attribute name="VALUE" x="39.497" y="163.0426" size="1.778" layer="96" rot="MR0"/>
-</instance>
 <instance part="C11" gate="G$1" x="35.56" y="165.1" rot="MR0"/>
 <instance part="P+5" gate="VCC" x="48.26" y="50.8" smashed="yes">
@@
 <instance part="P+11" gate="VCC" x="86.36" y="246.38"/>
 <instance part="C28" gate="G$1" x="93.98" y="215.9"/>
-<instance part="JP7" gate="A" x="60.96" y="238.76" rot="R90"/>
 <instance part="D3" gate="G$1" x="63.5" y="248.92" rot="R270"/>
 <instance part="P+10" gate="1" x="58.42" y="200.66" rot="MR0"/>
@@
 <instance part="ANALOG_LDO" gate="G$1" x="101.6" y="165.1"/>
 <instance part="C16" gate="G$1" x="119.38" y="152.4"/>
-<instance part="JP1" gate="A" x="86.36" y="175.26" rot="R90"/>
 <instance part="D1" gate="G$1" x="88.9" y="185.42" rot="R270"/>
 <instance part="P+14" gate="1" x="157.48" y="66.04" rot="MR0"/>
@@
 </instance>
 <instance part="GND12" gate="1" x="127" y="96.52"/>
+<instance part="JP1" gate="A" x="25.4" y="172.72"/>
+<instance part="GND13" gate="1" x="27.94" y="167.64"/>
 </instances>
 <busses>
@@
 <pinref part="R13" gate="G$1" pin="1"/>
 <wire x1="43.18" y1="124.46" x2="38.1" y2="124.46" width="0.1524" layer="91"/>
+<junction x="38.1" y="114.3"/>
+<junction x="38.1" y="124.46"/>
 </segment>
 <segment>
@@
 <junction x="127" y="111.76"/>
 </segment>
+<segment>
+<pinref part="JP1" gate="A" pin="2"/>
+<pinref part="GND13" gate="1" pin="GND"/>
+</segment>
 </net>
 <net name="AGND" class="0">
@@
 <pinref part="AGND1" gate="VR1" pin="AGND"/>
 <wire x1="33.02" y1="160.02" x2="25.4" y2="160.02" width="0.1524" layer="91"/>
-<pinref part="C10" gate="G$1" pin="-"/>
-<wire x1="33.02" y1="160.02" x2="40.64" y2="160.02" width="0.1524" layer="91"/>
+<pinref part="C11" gate="G$1" pin="2"/>
+<wire x1="33.02" y1="160.02" x2="35.56" y2="160.02" width="0.1524" layer="91"/>
+<junction x="33.02" y="160.02"/>
 </segment>
 <segment>
@@
 <wire x1="30.48" y1="167.64" x2="35.56" y2="167.64" width="0.1524" layer="91"/>
 <pinref part="VDD1" gate="G$1" pin="VDD"/>
-<pinref part="C10" gate="G$1" pin="+"/>
-<junction x="40.64" y="167.64"/>
 <pinref part="C11" gate="G$1" pin="1"/>
 <junction x="35.56" y="167.64"/>
@@
 <net name="N$32" class="0">
 <segment>
-<wire x1="63.5" y1="238.76" x2="63.5" y2="233.68" width="0.1524" layer="91"/>
+<wire x1="63.5" y1="246.38" x2="63.5" y2="233.68" width="0.1524" layer="91"/>
 <wire x1="63.5" y1="233.68" x2="63.5" y2="228.6" width="0.1524" layer="91"/>
 <wire x1="63.5" y1="228.6" x2="63.5" y2="218.44" width="0.1524" layer="91"/>
@@
 <pinref part="DIGITAL_LDO" gate="G$1" pin="SD/"/>
 <pinref part="C26" gate="G$1" pin="1"/>
-<pinref part="JP7" gate="A" pin="1"/>
+<pinref part="D3" gate="G$1" pin="C"/>
 </segment>
 </net>
@@
 </segment>
 </net>
-<net name="N$20" class="0">
-<segment>
-<wire x1="63.5" y1="241.3" x2="63.5" y2="246.38" width="0.1524" layer="91"/>
-<pinref part="JP7" gate="A" pin="2"/>
-<pinref part="D3" gate="G$1" pin="C"/>
-</segment>
-</net>
 <net name="N$21" class="0">
 <segment>
-<wire x1="88.9" y1="175.26" x2="88.9" y2="170.18" width="0.1524" layer="91"/>
+<wire x1="88.9" y1="182.88" x2="88.9" y2="170.18" width="0.1524" layer="91"/>
 <wire x1="88.9" y1="170.18" x2="88.9" y2="165.1" width="0.1524" layer="91"/>
 <wire x1="88.9" y1="165.1" x2="88.9" y2="154.94" width="0.1524" layer="91"/>
@@
 <pinref part="ANALOG_LDO" gate="G$1" pin="SD/"/>
 <pinref part="C14" gate="G$1" pin="1"/>
-<pinref part="JP1" gate="A" pin="1"/>
-</segment>
-</net>
-<net name="N$22" class="0">
-<segment>
-<wire x1="88.9" y1="177.8" x2="88.9" y2="182.88" width="0.1524" layer="91"/>
-<pinref part="JP1" gate="A" pin="2"/>
 <pinref part="D1" gate="G$1" pin="C"/>
 </segment>
@@
 <segment>
 <wire x1="78.74" y1="193.04" x2="73.66" y2="193.04" width="0.1524" layer="91"/>
-<wire x1="78.74" y1="193.04" x2="83.82" y2="193.04" width="0.1524" layer="91"/>
-<wire x1="83.82" y1="193.04" x2="83.82" y2="190.5" width="0.1524" layer="91"/>
 <junction x="73.66" y="193.04"/>
 <junction x="78.74" y="193.04"/>
@@
 <pinref part="C33" gate="G$1" pin="+"/>
 <pinref part="C34" gate="G$1" pin="1"/>
-<wire x1="83.82" y1="190.5" x2="88.9" y2="190.5" width="0.1524" layer="91"/>
+<wire x1="78.74" y1="193.04" x2="88.9" y2="193.04" width="0.1524" layer="91"/>
 <pinref part="D1" gate="G$1" pin="A"/>
-<wire x1="88.9" y1="190.5" x2="88.9" y2="187.96" width="0.1524" layer="91"/>
+<wire x1="88.9" y1="193.04" x2="88.9" y2="187.96" width="0.1524" layer="91"/>
 </segment>
 </net>
@@
 </segment>
 </net>
+<net name="N$20" class="0">
+<segment>
+<pinref part="U1" gate="AN_POWER" pin="VBAT"/>
+<pinref part="JP1" gate="A" pin="1"/>
+</segment>
+</net>

Commit message: v0.5
Parts:
- added JP2: (no value), jumper:JP1E
- added JP3, JP4: (no value), jumper:JP4E
Connections:
- net GND: now also JP2.2
- net PC0: now also JP3.4
- net PC1: now also JP3.3
- net PC2: now also JP3.2
- net PC3: now also JP3.1
- net PC4: now also JP4.4
- net PC5: now also JP4.3
- net VCC: now also JP2.1
Changed lines of the file:
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@@
 <layer number="96" name="Values" color="7" fill="1" visible="yes" active="yes"/>
 <layer number="97" name="Info" color="7" fill="1" visible="yes" active="yes"/>
-<layer number="98" name="Guide" color="6" fill="1" visible="yes" active="yes"/>
+<layer number="98" name="Guide" color="6" fill="1" visible="no" active="yes"/>
 <layer number="100" name="Muster" color="7" fill="1" visible="no" active="no"/>
-<layer number="101" name="Patch_Top" color="12" fill="4" visible="yes" active="yes"/>
-<layer number="116" name="Patch_BOT" color="9" fill="4" visible="yes" active="yes"/>
+<layer number="101" name="Patch_Top" color="12" fill="4" visible="no" active="yes"/>
+<layer number="116" name="Patch_BOT" color="9" fill="4" visible="no" active="yes"/>
 <layer number="200" name="200bmp" color="1" fill="10" visible="no" active="no"/>
 <layer number="201" name="201bmp" color="2" fill="1" visible="no" active="no"/>
@@
 <layer number="250" name="Descript" color="3" fill="1" visible="no" active="no"/>
 <layer number="251" name="SMDround" color="12" fill="11" visible="no" active="no"/>
-<layer number="254" name="cooling" color="7" fill="1" visible="yes" active="yes"/>
+<layer number="254" name="cooling" color="7" fill="1" visible="no" active="yes"/>
 </layers>
 <schematic xreflabel="%F%N/%S.%C%R" xrefpart="/%S.%C%R">
@@
 <part name="JP1" library="jumper" deviceset="JP1E" device=""/>
 <part name="GND13" library="supply1" deviceset="GND" device=""/>
+<part name="JP2" library="jumper" deviceset="JP1E" device=""/>
+<part name="P+15" library="supply1" deviceset="VCC" device=""/>
+<part name="GND14" library="supply1" deviceset="GND" device=""/>
+<part name="JP3" library="jumper" deviceset="JP4E" device=""/>
+<part name="JP4" library="jumper" deviceset="JP4E" device=""/>
 </parts>
 <sheets>
@@
 <instance part="JP1" gate="A" x="25.4" y="172.72"/>
 <instance part="GND13" gate="1" x="27.94" y="167.64"/>
+<instance part="JP2" gate="A" x="86.36" y="256.54"/>
+<instance part="P+15" gate="VCC" x="81.28" y="256.54" rot="MR0"/>
+<instance part="GND14" gate="1" x="93.98" y="256.54" rot="MR180"/>
+<instance part="JP3" gate="G$1" x="152.4" y="116.84" rot="R90"/>
+<instance part="JP4" gate="G$1" x="149.86" y="106.68" rot="R90"/>
 </instances>
 <busses>
@@
 <wire x1="86.36" y1="106.68" x2="104.14" y2="106.68" width="0.1524" layer="91"/>
 </segment>
+<segment>
+<pinref part="JP2" gate="A" pin="1"/>
+<pinref part="P+15" gate="VCC" pin="VCC"/>
+<wire x1="81.28" y1="254" x2="86.36" y2="254" width="0.1524" layer="91"/>
+</segment>
 </net>
 <net name="GND" class="0">
@@
 <pinref part="GND13" gate="1" pin="GND"/>
 </segment>
+<segment>
+<pinref part="JP2" gate="A" pin="2"/>
+<pinref part="GND14" gate="1" pin="GND"/>
+<wire x1="93.98" y1="254" x2="88.9" y2="254" width="0.1524" layer="91"/>
+</segment>
 </net>
 <net name="AGND" class="0">
@@
 <segment>
 <pinref part="U1" gate="PORTC_L" pin="PC0"/>
-<label x="154.94" y="121.92" size="1.27" layer="95" rot="MR0" xref="yes"/>
+<label x="144.78" y="121.92" size="1.27" layer="95" rot="MR0" xref="yes"/>
 <wire x1="154.94" y1="121.92" x2="160.02" y2="121.92" width="0.1524" layer="91"/>
+<pinref part="JP3" gate="G$1" pin="4"/>
 </segment>
 </net>
@@
 <segment>
 <pinref part="U1" gate="PORTC_L" pin="PC1"/>
-<label x="154.94" y="119.38" size="1.27" layer="95" rot="MR0" xref="yes"/>
+<label x="144.78" y="119.38" size="1.27" layer="95" rot="MR0" xref="yes"/>
 <wire x1="154.94" y1="119.38" x2="160.02" y2="119.38" width="0.1524" layer="91"/>
+<pinref part="JP3" gate="G$1" pin="3"/>
 </segment>
 </net>
@@
 <segment>
 <pinref part="U1" gate="PORTC_L" pin="PC2"/>
-<label x="154.94" y="116.84" size="1.27" layer="95" rot="MR0" xref="yes"/>
+<label x="144.78" y="116.84" size="1.27" layer="95" rot="MR0" xref="yes"/>
 <wire x1="154.94" y1="116.84" x2="160.02" y2="116.84" width="0.1524" layer="91"/>
+<pinref part="JP3" gate="G$1" pin="2"/>
 </segment>
 </net>
@@
 <segment>
 <pinref part="U1" gate="PORTC_L" pin="PC3"/>
-<label x="154.94" y="114.3" size="1.27" layer="95" rot="MR0" xref="yes"/>
+<label x="144.78" y="114.3" size="1.27" layer="95" rot="MR0" xref="yes"/>
 <wire x1="154.94" y1="114.3" x2="160.02" y2="114.3" width="0.1524" layer="91"/>
+<pinref part="JP3" gate="G$1" pin="1"/>
 </segment>
 </net>
@@
 <segment>
 <pinref part="U1" gate="PORTC_L" pin="PC4"/>
-<label x="154.94" y="111.76" size="1.27" layer="95" rot="MR0" xref="yes"/>
-<wire x1="154.94" y1="111.76" x2="160.02" y2="111.76" width="0.1524" layer="91"/>
+<label x="144.78" y="111.76" size="1.27" layer="95" rot="MR0" xref="yes"/>
+<wire x1="152.4" y1="111.76" x2="160.02" y2="111.76" width="0.1524" layer="91"/>
+<pinref part="JP4" gate="G$1" pin="4"/>
 </segment>
 </net>
@@
 <segment>
 <pinref part="U1" gate="PORTC_L" pin="PC5"/>
-<label x="154.94" y="109.22" size="1.27" layer="95" rot="MR0" xref="yes"/>
-<wire x1="154.94" y1="109.22" x2="160.02" y2="109.22" width="0.1524" layer="91"/>
+<label x="144.78" y="109.22" size="1.27" layer="95" rot="MR0" xref="yes"/>
+<wire x1="152.4" y1="109.22" x2="160.02" y2="109.22" width="0.1524" layer="91"/>
+<pinref part="JP4" gate="G$1" pin="3"/>
 </segment>
 </net>
@@
 <segment>
 <pinref part="U1" gate="PORTC_L" pin="PC6"/>
-<label x="154.94" y="106.68" size="1.27" layer="95" rot="MR0" xref="yes"/>
+<label x="144.78" y="106.68" size="1.27" layer="95" rot="MR0" xref="yes"/>
 <wire x1="154.94" y1="106.68" x2="160.02" y2="106.68" width="0.1524" layer="91"/>
 </segment>
@@
 <segment>
 <pinref part="U1" gate="PORTC_L" pin="PC7"/>
-<label x="154.94" y="104.14" size="1.27" layer="95" rot="MR0" xref="yes"/>
+<label x="144.78" y="104.14" size="1.27" layer="95" rot="MR0" xref="yes"/>
 <wire x1="154.94" y1="104.14" x2="160.02" y2="104.14" width="0.1524" layer="91"/>
 </segment>
