File: narsil.sch (EAGLE design)
At the start: 79 parts, among them Q1 IRLML5203, Q5 IRLML5203, U1 STM32F10XRXT6, X1 PN61729-S

Commit message: v0.6
Parts:
- added C21, C22: (no value), resistor:C-EUC0805
- added Q2: 32kHz, crystal:MC146
- added R/C3: (no value), resistor:R-EU_M0805
Connections:
- new net N$22: R/C3.2, U1PORTD/OSC.PD1/OSC=>
- net GND: now also C21.1, C22.1
- net N$4: now also R/C3.1; no longer U1PORTD/OSC.PD1/OSC=>
- net PC14: now also C21.2, Q2G$1.1; no longer BTN_1.S, BTN_1.S1, C43.2, R36.2
- net PC15: now also C22.2, Q2G$1.2; no longer BTN_2.S, BTN_2.S1, C42.2, R35.2
- net PC6: now also BTN_2.S, BTN_2.S1, C42.2, R35.2
- net PC7: now also BTN_1.S, BTN_1.S1, C43.2, R36.2
Other:
- moved on the sheet: C5, C6, QF1
Changed lines of the file:
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@@
 <part name="JP3" library="jumper" deviceset="JP4E" device=""/>
 <part name="JP4" library="jumper" deviceset="JP4E" device=""/>
+<part name="R/C3" library="resistor" deviceset="R-EU_" device="M0805"/>
+<part name="Q2" library="crystal" deviceset="MC146" device="" value="32kHz"/>
+<part name="C21" library="resistor" deviceset="C-EU" device="C0805"/>
+<part name="GND17" library="supply1" deviceset="GND" device=""/>
+<part name="C22" library="resistor" deviceset="C-EU" device="C0805"/>
 </parts>
 <sheets>
@@
 <instance part="C4" gate="G$1" x="35.56" y="238.76" rot="MR90"/>
 <instance part="GND5" gate="1" x="40.64" y="236.22" rot="MR0"/>
-<instance part="QF1" gate="G$1" x="33.02" y="187.96" smashed="yes" rot="R90">
-<attribute name="NAME" x="32.004" y="190.5" size="1.778" layer="95" rot="R90"/>
-<attribute name="VALUE" x="35.56" y="190.5" size="1.778" layer="96"/>
-</instance>
-<instance part="C5" gate="G$1" x="33.02" y="195.58"/>
-<instance part="C6" gate="G$1" x="33.02" y="180.34" rot="R180"/>
+<instance part="QF1" gate="G$1" x="35.56" y="187.96" smashed="yes" rot="R90">
+<attribute name="NAME" x="34.544" y="190.5" size="1.778" layer="95" rot="R90"/>
+<attribute name="VALUE" x="38.1" y="190.5" size="1.778" layer="96"/>
+</instance>
+<instance part="C5" gate="G$1" x="35.56" y="195.58"/>
+<instance part="C6" gate="G$1" x="35.56" y="180.34" rot="R180"/>
 <instance part="GND6" gate="1" x="40.64" y="175.26"/>
 <instance part="APWR" gate="G$1" x="99.06" y="241.3"/>
@@
 <instance part="JP3" gate="G$1" x="152.4" y="116.84" rot="R90"/>
 <instance part="JP4" gate="G$1" x="149.86" y="106.68" rot="R90"/>
+<instance part="R/C3" gate="G$1" x="30.48" y="185.42" rot="MR0"/>
+<instance part="Q2" gate="G$1" x="137.16" y="78.74" rot="MR270"/>
+<instance part="C21" gate="G$1" x="132.08" y="81.28" rot="MR270"/>
+<instance part="GND17" gate="1" x="129.54" y="73.66" rot="MR0"/>
+<instance part="C22" gate="G$1" x="132.08" y="76.2" rot="MR270"/>
 </instances>
 <busses>
@@
 <segment>
 <pinref part="QF1" gate="G$1" pin="2"/>
-<wire x1="38.1" y1="187.96" x2="40.64" y2="187.96" width="0.1524" layer="91"/>
 <wire x1="40.64" y1="187.96" x2="40.64" y2="177.8" width="0.1524" layer="91"/>
 <pinref part="C6" gate="G$1" pin="1"/>
-<wire x1="33.02" y1="177.8" x2="40.64" y2="177.8" width="0.1524" layer="91"/>
+<wire x1="35.56" y1="177.8" x2="40.64" y2="177.8" width="0.1524" layer="91"/>
 <pinref part="C5" gate="G$1" pin="1"/>
-<wire x1="33.02" y1="198.12" x2="40.64" y2="198.12" width="0.1524" layer="91"/>
+<wire x1="35.56" y1="198.12" x2="40.64" y2="198.12" width="0.1524" layer="91"/>
 <wire x1="40.64" y1="198.12" x2="40.64" y2="187.96" width="0.1524" layer="91"/>
 <pinref part="GND6" gate="1" pin="GND"/>
@@
 <wire x1="93.98" y1="254" x2="88.9" y2="254" width="0.1524" layer="91"/>
 </segment>
+<segment>
+<junction x="129.54" y="76.2"/>
+<pinref part="C21" gate="G$1" pin="1"/>
+<pinref part="GND17" gate="1" pin="GND"/>
+<pinref part="C22" gate="G$1" pin="1"/>
+<wire x1="129.54" y1="76.2" x2="129.54" y2="81.28" width="0.1524" layer="91"/>
+</segment>
 </net>
 <net name="AGND" class="0">
@@
 <pinref part="U1" gate="PORTD/OSC" pin="PD0/OSC&lt;="/>
 <wire x1="25.4" y1="187.96" x2="25.4" y2="190.5" width="0.1524" layer="91"/>
-<wire x1="25.4" y1="190.5" x2="33.02" y2="190.5" width="0.1524" layer="91"/>
-<junction x="33.02" y="190.5"/>
+<wire x1="25.4" y1="190.5" x2="35.56" y2="190.5" width="0.1524" layer="91"/>
+<junction x="35.56" y="190.5"/>
 </segment>
 </net>
@@
 <pinref part="QF1" gate="G$1" pin="1"/>
 <pinref part="C6" gate="G$1" pin="2"/>
-<pinref part="U1" gate="PORTD/OSC" pin="PD1/OSC=&gt;"/>
-<wire x1="25.4" y1="185.42" x2="33.02" y2="185.42" width="0.1524" layer="91"/>
-<junction x="33.02" y="185.42"/>
+<pinref part="R/C3" gate="G$1" pin="1"/>
+<junction x="35.56" y="185.42"/>
 </segment>
 </net>
@@
 <wire x1="154.94" y1="106.68" x2="160.02" y2="106.68" width="0.1524" layer="91"/>
 </segment>
+<segment>
+<pinref part="C42" gate="G$1" pin="2"/>
+<wire x1="109.22" y1="78.74" x2="106.68" y2="78.74" width="0.1524" layer="91"/>
+<wire x1="106.68" y1="78.74" x2="106.68" y2="81.28" width="0.1524" layer="91"/>
+<label x="106.68" y="81.28" size="1.27" layer="95" rot="R90" xref="yes"/>
+<pinref part="R35" gate="G$1" pin="2"/>
+<wire x1="106.68" y1="78.74" x2="106.68" y2="71.12" width="0.1524" layer="91"/>
+<pinref part="BTN_2" gate="G$1" pin="S1"/>
+<wire x1="106.68" y1="71.12" x2="106.68" y2="68.58" width="0.1524" layer="91"/>
+<wire x1="109.22" y1="71.12" x2="106.68" y2="71.12" width="0.1524" layer="91"/>
+<pinref part="BTN_2" gate="G$1" pin="S"/>
+<wire x1="109.22" y1="68.58" x2="106.68" y2="68.58" width="0.1524" layer="91"/>
+</segment>
 </net>
 <net name="PC7" class="0">
@@
 <label x="144.78" y="104.14" size="1.27" layer="95" rot="MR0" xref="yes"/>
 <wire x1="154.94" y1="104.14" x2="160.02" y2="104.14" width="0.1524" layer="91"/>
+</segment>
+<segment>
+<pinref part="C43" gate="G$1" pin="2"/>
+<wire x1="88.9" y1="78.74" x2="86.36" y2="78.74" width="0.1524" layer="91"/>
+<wire x1="86.36" y1="78.74" x2="86.36" y2="81.28" width="0.1524" layer="91"/>
+<label x="86.36" y="81.28" size="1.27" layer="95" rot="R90" xref="yes"/>
+<pinref part="R36" gate="G$1" pin="2"/>
+<wire x1="86.36" y1="78.74" x2="86.36" y2="71.12" width="0.1524" layer="91"/>
+<pinref part="BTN_1" gate="G$1" pin="S1"/>
+<wire x1="86.36" y1="71.12" x2="86.36" y2="68.58" width="0.1524" layer="91"/>
+<wire x1="88.9" y1="71.12" x2="86.36" y2="71.12" width="0.1524" layer="91"/>
+<pinref part="BTN_1" gate="G$1" pin="S"/>
+<wire x1="88.9" y1="68.58" x2="86.36" y2="68.58" width="0.1524" layer="91"/>
 </segment>
 </net>
@@
 <pinref part="U1" gate="PORTC_H" pin="PC14"/>
 <label x="154.94" y="81.28" size="1.27" layer="95" rot="MR0" xref="yes"/>
-<wire x1="154.94" y1="81.28" x2="160.02" y2="81.28" width="0.1524" layer="91"/>
-</segment>
-<segment>
-<wire x1="88.9" y1="68.58" x2="86.36" y2="68.58" width="0.1524" layer="91"/>
-<wire x1="88.9" y1="71.12" x2="86.36" y2="71.12" width="0.1524" layer="91"/>
-<wire x1="86.36" y1="71.12" x2="86.36" y2="68.58" width="0.1524" layer="91"/>
-<wire x1="86.36" y1="68.58" x2="86.36" y2="78.74" width="0.1524" layer="91"/>
-<wire x1="86.36" y1="78.74" x2="86.36" y2="81.28" width="0.1524" layer="91"/>
-<wire x1="88.9" y1="78.74" x2="86.36" y2="78.74" width="0.1524" layer="91"/>
-<junction x="86.36" y="68.58"/>
-<junction x="86.36" y="78.74"/>
-<pinref part="C43" gate="G$1" pin="2"/>
-<pinref part="R36" gate="G$1" pin="2"/>
-<pinref part="BTN_1" gate="G$1" pin="S"/>
-<pinref part="BTN_1" gate="G$1" pin="S1"/>
-<label x="86.36" y="81.28" size="1.27" layer="95" rot="R90" xref="yes"/>
+<wire x1="160.02" y1="81.28" x2="139.7" y2="81.28" width="0.1524" layer="91"/>
+<wire x1="139.7" y1="81.28" x2="139.7" y2="83.82" width="0.1524" layer="91"/>
+<pinref part="C21" gate="G$1" pin="2"/>
+<pinref part="Q2" gate="G$1" pin="1"/>
+<wire x1="137.16" y1="81.28" x2="139.7" y2="81.28" width="0.1524" layer="91"/>
+<junction x="137.16" y="81.28"/>
 </segment>
 </net>
@@
 <pinref part="U1" gate="PORTC_H" pin="PC15"/>
 <label x="154.94" y="78.74" size="1.27" layer="95" rot="MR0" xref="yes"/>
-<wire x1="154.94" y1="78.74" x2="160.02" y2="78.74" width="0.1524" layer="91"/>
-</segment>
-<segment>
-<wire x1="109.22" y1="68.58" x2="106.68" y2="68.58" width="0.1524" layer="91"/>
-<wire x1="109.22" y1="71.12" x2="106.68" y2="71.12" width="0.1524" layer="91"/>
-<wire x1="106.68" y1="71.12" x2="106.68" y2="68.58" width="0.1524" layer="91"/>
-<wire x1="106.68" y1="68.58" x2="106.68" y2="78.74" width="0.1524" layer="91"/>
-<wire x1="106.68" y1="78.74" x2="106.68" y2="81.28" width="0.1524" layer="91"/>
-<wire x1="109.22" y1="78.74" x2="106.68" y2="78.74" width="0.1524" layer="91"/>
-<junction x="106.68" y="68.58"/>
-<junction x="106.68" y="78.74"/>
-<pinref part="C42" gate="G$1" pin="2"/>
-<pinref part="R35" gate="G$1" pin="2"/>
-<pinref part="BTN_2" gate="G$1" pin="S"/>
-<pinref part="BTN_2" gate="G$1" pin="S1"/>
-<label x="106.68" y="81.28" size="1.27" layer="95" rot="R90" xref="yes"/>
+<wire x1="160.02" y1="78.74" x2="142.24" y2="78.74" width="0.1524" layer="91"/>
+<wire x1="142.24" y1="78.74" x2="142.24" y2="76.2" width="0.1524" layer="91"/>
+<pinref part="C22" gate="G$1" pin="2"/>
+<pinref part="Q2" gate="G$1" pin="2"/>
+<wire x1="137.16" y1="76.2" x2="142.24" y2="76.2" width="0.1524" layer="91"/>
+<junction x="137.16" y="76.2"/>
 </segment>
 </net>
@@
 </segment>
 </net>
+<net name="N$22" class="0">
+<segment>
+<pinref part="U1" gate="PORTD/OSC" pin="PD1/OSC=&gt;"/>
+<pinref part="R/C3" gate="G$1" pin="2"/>
+</segment>
+</net>
